Commit message: 1

File: src/myagv/myagv/urdf/mecanum_properties.urdf.xacro (robot description, xacro)
@@ -5,7 +5,5 @@
   <xacro:property name="base_height" value="0.08" />
   <xacro:property name="base_mass" value="3.02" />
-  <!-- set empty on the wheel_mesh_file to use geometry instead of mesh -->
   <xacro:property name="base_mesh_file" value="" />
-  <!-- <xacro:property name="base_mesh_file" value="file://$(find myagv_description)/meshes/base.dae" /> -->
   <xacro:property name="wheel_radius" value="0.04" />
   <xacro:property name="wheel_width" value="0.03" />
@@ -15,7 +13,5 @@
   <xacro:property name="wheel_mass" value="0.6" />
   <xacro:property name="wheel_torque" value="20" />
-  <!-- set empty on the wheel_mesh_file to use geometry instead of mesh -->
   <xacro:property name="wheel_mesh_file" value="" />
-  <!-- <xacro:property name="wheel_mesh_file" value="file://$(find myagv_description)/meshes/tire.dae" /> -->
   <xacro:property name="laser_pose">
     <origin xyz="0.04 0 0.05" rpy="0 0 0"/>

File: src/myagv/myagv/urdf/mech/base.urdf.xacro (robot description, xacro)
@@ -1,5 +1,5 @@
 <?xml version="1.0"?>
 <robot xmlns:xacro="http://ros.org/wiki/xacro">
-  <xacro:macro name="base" params="length width height mass wheel_radius wheel_pos_z mesh_file">
+  <xacro:macro name="base" params="length width height mass wheel_radius wheel_pos_z ">
     <link name="base_footprint"/>
     <link name="base_link">
@@ -7,10 +7,6 @@
         <origin xyz="0 0 0" rpy="0 0 0"/>
         <geometry>
-          <xacro:if value="${mesh_file == ''}">
-            <box size="${length} ${width} ${height}"/>
-          </xacro:if>
-          <xacro:unless value="${mesh_file == ''}">
-            <mesh filename="${mesh_file}" scale="1 1 1"/>
-          </xacro:unless>
+          <!-- Always use box -->
+          <box size="${length} ${width} ${height}"/>
         </geometry>
         <material name="purple">

File: src/myagv/myagv/urdf/mech/mecanum_wheel.urdf.xacro (robot description, xacro)
@@ -1,18 +1,14 @@
 <?xml version="1.0"?>
 <robot xmlns:xacro="http://ros.org/wiki/xacro" xmlns:gz="http://gazebosim.org/schema">
-  <xacro:macro name="mecanum_wheel" params="side radius width pos_x pos_y pos_z mass mesh_file">
+  <xacro:macro name="mecanum_wheel" params="side radius width pos_x pos_y pos_z mass ">
     <link name="${side}_wheel_link">
       <visual>
         <origin xyz="0 0 0" rpy="${pi/2} 0 0"/>
         <geometry>
-          <xacro:if value="${mesh_file == ''}">
-            <cylinder radius="${radius}" length="${width}"/>
-          </xacro:if>
-          <xacro:unless value="${mesh_file == ''}">
-            <mesh filename="${mesh_file}" scale="1 1 1"/>
-          </xacro:unless>
+          <!-- Always use cylinder for the wheel -->
+          <cylinder radius="${radius}" length="${width}"/>
         </geometry>
         <material name="blue">
-            <color rgba="0.1764 0.4588 0.8509 1.0"/>
+          <color rgba="0.1764 0.4588 0.8509 1.0"/>
         </material>
       </visual>
@@ -38,6 +34,5 @@
               <mu>1.5</mu>
               <mu2>0.7</mu2>
-              <kp>200000.0</kp>
-              <kd>5000.0</kd>
+              <!-- kp/kd removed to avoid SDF warnings -->
               <xacro:if value="${side == 'front_left'}">
                 <fdir1 gz:expressed_in="base_footprint">1 -1 0</fdir1>

File: src/myagv/myagv/urdf/robots/core.urdf.xacro (robot description, xacro)
@@ -1,12 +1,11 @@
 <?xml version="1.0"?>
 <robot name="myagv_mecanum" xmlns:xacro="http://ros.org/wiki/xacro">
-  <xacro:include filename="$(find myagv_description)/urdf/mecanum_properties.urdf.xacro" />
-  <xacro:include filename="$(find myagv_description)/urdf/mech/base.urdf.xacro" />
-  <xacro:include filename="$(find myagv_description)/urdf/mech/mecanum_wheel.urdf.xacro" />
-  <xacro:include filename="$(find myagv_description)/urdf/sensors/plugins.urdf.xacro" />
-  <xacro:include filename="$(find myagv_description)/urdf/sensors/imu.urdf.xacro" />
-  <xacro:include filename="$(find myagv_description)/urdf/sensors/generic_laser.urdf.xacro" />
-  <!-- <xacro:include filename="$(find myagv_description)/urdf/sensors/depth_sensor.urdf.xacro" /> -->
-  <xacro:include filename="$(find myagv_description)/urdf/controllers/omni_drive.urdf.xacro" />
+  <xacro:include filename="$(find myagv)/urdf/mecanum_properties.urdf.xacro" />
+  <xacro:include filename="$(find myagv)/urdf/mech/base.urdf.xacro" />
+  <xacro:include filename="$(find myagv)/urdf/mech/mecanum_wheel.urdf.xacro" />
+  <xacro:include filename="$(find myagv)/urdf/sensors/plugins.urdf.xacro" />
+  <xacro:include filename="$(find myagv)/urdf/sensors/imu.urdf.xacro" />
+  <xacro:include filename="$(find myagv)/urdf/sensors/generic_laser.urdf.xacro" />
+  <xacro:include filename="$(find myagv)/urdf/controllers/omni_drive.urdf.xacro" />
   <xacro:base
     length="${base_length}"
@@ -16,5 +15,4 @@
     wheel_radius="${wheel_radius}"
     wheel_pos_z="${wheel_pos_z}"
-    mesh_file="${base_mesh_file}"
   />
   <xacro:mecanum_wheel
@@ -26,5 +24,4 @@
     pos_z="${wheel_pos_z}"
     mass="${wheel_mass}"
-    mesh_file="${wheel_mesh_file}"
   />
   <xacro:mecanum_wheel
@@ -36,5 +33,4 @@
     pos_z="${wheel_pos_z}"
     mass="${wheel_mass}"
-    mesh_file="${wheel_mesh_file}"
   />
   <xacro:mecanum_wheel
@@ -46,5 +42,4 @@
     pos_z="${wheel_pos_z}"
     mass="${wheel_mass}"
-    mesh_file="${wheel_mesh_file}"
   />
   <xacro:mecanum_wheel
@@ -56,5 +51,4 @@
     pos_z="${wheel_pos_z}"
     mass="${wheel_mass}"
-    mesh_file="${wheel_mesh_file}"
   />
   <xacro:imu/>
@@ -62,7 +56,4 @@
     <xacro:insert_block name="laser_pose" />
   </xacro:generic_laser>
-  <!-- <xacro:depth_sensor>
-    <xacro:insert_block name="depth_sensor_pose" />
-  </xacro:depth_sensor> -->
   <xacro:omni_drive_controller
     wheel_separation="${wheel_pos_y * 2}"

File: src/myagv/myagv/urdf/sensors/generic_laser.urdf.xacro (robot description, xacro)
@@ -1,5 +1,5 @@
 <?xml version="1.0"?>
 <robot xmlns:xacro="http://ros.org/wiki/xacro">
-  <xacro:include filename="$(find myagv_description)/urdf/sensors/laser.urdf.xacro" />
+  <xacro:include filename="$(find myagv)/urdf/sensors/laser.urdf.xacro" />
   <xacro:macro name="generic_laser" params="*origin">
     <xacro:laser
